File: ALU.kicad_pcb (KiCad board)
At the start: 2 copper layers, 0 parts

Commit message: pcb layout start (attempt 3)
15.3 hours work time
Parts:
- added BT1: 3V0, Battery:Battery_Panasonic_CR2032-VS1N_Vertical_CircularHoles, F.Cu at (41.1, 79.6)
- added C1: 10u, Capacitor_THT:CP_Radial_D5.0mm_P2.00mm, F.Cu at (75.8, 72.5)
- added C10: 100n, Capacitor_SMD:C_0805_2012Metric, F.Cu at (53.4, 42.3)
- added C11: 100n, Capacitor_SMD:C_0805_2012Metric, F.Cu at (53.4, 45.3)
- added C12: 100n, Capacitor_SMD:C_0805_2012Metric, F.Cu at (57.8, 18.2)
- added C13: 100n, Capacitor_SMD:C_0805_2012Metric, F.Cu at (57.8, 21.2)
- added C14: 100n, Capacitor_SMD:C_0805_2012Metric, F.Cu at (57.8, 24.2)
- added C15: 100n, Capacitor_SMD:C_0805_2012Metric, F.Cu at (57.8, 27.2)
- added C16: 100n, Capacitor_SMD:C_0805_2012Metric, F.Cu at (57.8, 30.2)
- added C17: 100n, Capacitor_SMD:C_0805_2012Metric, F.Cu at (57.8, 33.3)
- added C18: 100n, Capacitor_SMD:C_0805_2012Metric, F.Cu at (57.8, 36.3)
- added C19: 100n, Capacitor_SMD:C_0805_2012Metric, F.Cu at (57.8, 39.3)
- added C2: 100n, Capacitor_SMD:C_0805_2012Metric, F.Cu at (53.4, 18.2)
- added C20: 100n, Capacitor_SMD:C_0805_2012Metric, F.Cu at (57.8, 42.3)
- added C21: 100n, Capacitor_SMD:C_0805_2012Metric, F.Cu at (57.8, 45.3)
- added C22: 100n, Capacitor_SMD:C_0805_2012Metric, F.Cu at (62.3, 18.2)
- added C23: 100n, Capacitor_SMD:C_0805_2012Metric, F.Cu at (62.3, 21.2)
- added C24: 100n, Capacitor_SMD:C_0805_2012Metric, F.Cu at (62.3, 24.2)
- added C25: 100n, Capacitor_SMD:C_0805_2012Metric, F.Cu at (62.3, 27.2)
- added C26: 100n, Capacitor_SMD:C_0805_2012Metric, F.Cu at (62.3, 30.2)
- added C27: 100n, Capacitor_SMD:C_0805_2012Metric, F.Cu at (62.3, 33.3)
- added C28: 100n, Capacitor_SMD:C_0805_2012Metric, F.Cu at (62.3, 36.3)
- added C29: 100n, Capacitor_SMD:C_0805_2012Metric, F.Cu at (62.3, 39.3)
- added C3: 100n, Capacitor_SMD:C_0805_2012Metric, F.Cu at (53.4, 21.2)
- added C30: 100n, Capacitor_SMD:C_0805_2012Metric, F.Cu at (62.3, 42.3)
- added C31: 100n, Capacitor_SMD:C_0805_2012Metric, F.Cu at (62.3, 45.3)
- added C32: 100n, Capacitor_SMD:C_0805_2012Metric, F.Cu at (66.7, 18.2)
- added C33: 100n, Capacitor_SMD:C_0805_2012Metric, F.Cu at (66.7, 21.2)
- added C34: 100n, Capacitor_SMD:C_0805_2012Metric, F.Cu at (66.7, 24.2)
- added C35: 100n, Capacitor_SMD:C_0805_2012Metric, F.Cu at (66.7, 27.2)
- added C36: 100n, Capacitor_SMD:C_0805_2012Metric, F.Cu at (66.7, 30.2)
- added C37: 100n, Capacitor_SMD:C_0805_2012Metric, F.Cu at (66.7, 33.3)
- added C38: 100n, Capacitor_SMD:C_0805_2012Metric, F.Cu at (66.7, 36.3)
- added C39: 100n, Capacitor_SMD:C_0805_2012Metric, F.Cu at (66.7, 39.3)
- added C4: 100n, Capacitor_SMD:C_0805_2012Metric, F.Cu at (53.4, 24.2)
- added C40: 100n, Capacitor_SMD:C_0805_2012Metric, F.Cu at (66.7, 42.3)
- added C41: 100n, Capacitor_SMD:C_0805_2012Metric, F.Cu at (66.7, 45.3)
- added C42: 100n, Capacitor_SMD:C_0805_2012Metric, F.Cu at (71.2, 18.2)
- added C43: 100n, Capacitor_SMD:C_0805_2012Metric, F.Cu at (71.2, 21.2)
- added C44: 100n, Capacitor_SMD:C_0805_2012Metric, F.Cu at (71.2, 24.2)
- added C45: 100n, Capacitor_SMD:C_0805_2012Metric, F.Cu at (71.2, 27.2)
- added C46: 100n, Capacitor_SMD:C_0805_2012Metric, F.Cu at (71.2, 30.2)
- added C47: 100n, Capacitor_SMD:C_0805_2012Metric, F.Cu at (71.2, 33.3)
- added C48: 100n, Capacitor_SMD:C_0805_2012Metric, F.Cu at (71.2, 36.3)
- added C49: 100n, Capacitor_SMD:C_0805_2012Metric, F.Cu at (71.2, 39.3)
- added C5: 100n, Capacitor_SMD:C_0805_2012Metric, F.Cu at (53.4, 27.2)
- added C50: 100n, Capacitor_SMD:C_0805_2012Metric, F.Cu at (71.2, 42.3)
- added C51: 100n, Capacitor_SMD:C_0805_2012Metric, F.Cu at (71.2, 45.3)
- added C52: 100n, Capacitor_SMD:C_0805_2012Metric, F.Cu at (75.6, 18.2)
- added C53: 100n, Capacitor_SMD:C_0805_2012Metric, F.Cu at (75.6, 21.2)
- added C54: 100n, Capacitor_SMD:C_0805_2012Metric, F.Cu at (75.6, 24.2)
- added C55: 100n, Capacitor_SMD:C_0805_2012Metric, F.Cu at (75.6, 27.2)
- added C57: 100n, Capacitor_SMD:C_0805_2012Metric, F.Cu at (75.6, 30.2)
- added C58: 100n, Capacitor_SMD:C_0805_2012Metric, F.Cu at (75.6, 33.3)
- added C59: 100n, Capacitor_SMD:C_0805_2012Metric, F.Cu at (75.6, 36.3)
- added C6: 100n, Capacitor_SMD:C_0805_2012Metric, F.Cu at (53.4, 30.2)
- added C60: 100n, Capacitor_SMD:C_0805_2012Metric, F.Cu at (75.6, 39.3)
- added C61: 100n, Capacitor_SMD:C_0805_2012Metric, F.Cu at (75.6, 42.3)
- added C7: 100n, Capacitor_SMD:C_0805_2012Metric, F.Cu at (53.4, 33.3)
- added C8: 100n, Capacitor_SMD:C_0805_2012Metric, F.Cu at (53.4, 36.3)
- added C9: 100n, Capacitor_SMD:C_0805_2012Metric, F.Cu at (53.4, 39.3)
- added D1: LED_GREEN, LED_SMD:LED_0805_2012Metric, F.Cu at (71.6, 51.6)
- added D10: LED_RED, LED_SMD:LED_0805_2012Metric, F.Cu at (76.1, 63.8)
- added D11: LED_YELLOW, LED_SMD:LED_0603_1608Metric, F.Cu at (75.5, 77.1)
- added D2: LED_GREEN, LED_SMD:LED_0805_2012Metric, F.Cu at (71.6, 54.7)
- added D3: LED_GREEN, LED_SMD:LED_0805_2012Metric, F.Cu at (71.6, 57.7)
- added D4: LED_GREEN, LED_SMD:LED_0805_2012Metric, F.Cu at (71.6, 60.8)
- added D5: LED_GREEN, LED_SMD:LED_0805_2012Metric, F.Cu at (71.6, 63.8)
- added D6: LED_GREEN, LED_SMD:LED_0805_2012Metric, F.Cu at (76.1, 51.6)
- added D7: LED_GREEN, LED_SMD:LED_0805_2012Metric, F.Cu at (76.1, 54.7)
- added D8: LED_GREEN, LED_SMD:LED_0805_2012Metric, F.Cu at (76.1, 57.7)
- added D9: LED_RED, LED_SMD:LED_0805_2012Metric, F.Cu at (76.1, 60.8)
- added R1: 10K, Resistor_SMD:R_0805_2012Metric, F.Cu at (19.7, 51.6)
- added R10: 10K, Resistor_SMD:R_0805_2012Metric, F.Cu at (24.1, 51.6)
- added R11: 10K, Resistor_SMD:R_0805_2012Metric, F.Cu at (24.1, 54.6)
- added R12: 10K, Resistor_SMD:R_0805_2012Metric, F.Cu at (24.1, 57.5)
- added R13: 10K, Resistor_SMD:R_0805_2012Metric, F.Cu at (24.1, 60.5)
- added R14: 10K, Resistor_SMD:R_0805_2012Metric, F.Cu at (24.1, 63.4)
- added R15: 10K, Resistor_SMD:R_0805_2012Metric, F.Cu at (24.1, 66.4)
- added R16: 10K, Resistor_SMD:R_0805_2012Metric, F.Cu at (24.1, 69.3)
- added R17: 10K, Resistor_SMD:R_0805_2012Metric, F.Cu at (24.1, 72.3)
- added R18: 10K, Resistor_SMD:R_0805_2012Metric, F.Cu at (24.1, 75.2)
- added R19: 10K, Resistor_SMD:R_0805_2012Metric, F.Cu at (28.5, 51.6)
- added R2: 10K, Resistor_SMD:R_0805_2012Metric, F.Cu at (19.7, 54.6)
- added R20: 10K, Resistor_SMD:R_0805_2012Metric, F.Cu at (28.5, 54.6)
- added R21: 10K, Resistor_SMD:R_0805_2012Metric, F.Cu at (28.5, 57.5)
- added R22: 10K, Resistor_SMD:R_0805_2012Metric, F.Cu at (28.5, 60.5)
- added R23: 680, Resistor_SMD:R_0805_2012Metric, F.Cu at (28.5, 63.4)
- added R24: 220, Resistor_SMD:R_0805_2012Metric, F.Cu at (28.5, 66.4)
- added R25: 220, Resistor_SMD:R_0805_2012Metric, F.Cu at (28.5, 69.3)
- added R26: 220, Resistor_SMD:R_0805_2012Metric, F.Cu at (28.5, 72.3)
- added R27: 220, Resistor_SMD:R_0805_2012Metric, F.Cu at (28.5, 75.2)
- added R28: 220, Resistor_SMD:R_0805_2012Metric, F.Cu at (32.9, 51.6)
- added R29: 220, Resistor_SMD:R_0805_2012Metric, F.Cu at (32.9, 54.6)
- added R3: 10K, Resistor_SMD:R_0805_2012Metric, F.Cu at (19.7, 57.5)
- added R30: 220, Resistor_SMD:R_0805_2012Metric, F.Cu at (32.9, 57.5)
- added R31: 220, Resistor_SMD:R_0805_2012Metric, F.Cu at (32.9, 60.5)
- added R32: 470, Resistor_SMD:R_0805_2012Metric, F.Cu at (32.9, 63.4)
- added R33: 470, Resistor_SMD:R_0805_2012Metric, F.Cu at (32.9, 66.4)
- added R4: 10K, Resistor_SMD:R_0805_2012Metric, F.Cu at (19.7, 60.5)
- added R5: 10K, Resistor_SMD:R_0805_2012Metric, F.Cu at (19.7, 63.4)
- added R6: 10K, Resistor_SMD:R_0805_2012Metric, F.Cu at (19.7, 66.4)
- added R7: 10K, Resistor_SMD:R_0805_2012Metric, F.Cu at (19.7, 69.3)
- added R8: 10K, Resistor_SMD:R_0805_2012Metric, F.Cu at (19.7, 72.3)
- added R9: 10K, Resistor_SMD:R_0805_2012Metric, F.Cu at (19.7, 75.2)
- added SW1: SW_DIP_x06, Button_Switch_THT:SW_DIP_SPSTx06_Slide_9.78x17.42mm_W7.62mm_P2.54mm, F.Cu at (59.9, 53.4)
- added SW2: SW_SPST, Button_Switch_THT:SW_DIP_SPSTx01_Slide_9.78x4.72mm_W7.62mm_P2.54mm, F.Cu at (19.4, 79.9)
- added SW3: SW_DIP_x08, Button_Switch_THT:SW_DIP_SPSTx08_Slide_9.78x22.5mm_W7.62mm_P2.54mm, F.Cu at (117.8, 40.3)
- added SW4: SW_DIP_x08, Button_Switch_THT:SW_DIP_SPSTx08_Slide_9.78x22.5mm_W7.62mm_P2.54mm, F.Cu at (131.1, 40.3)
- added U1: 74LVC2G86, Package_SO:VSSOP-8_2.3x2mm_P0.5mm, F.Cu at (20.3, 18.6)
- added U10: 74LVC2G08, Package_SO:VSSOP-8_2.3x2mm_P0.5mm, F.Cu at (25.9, 18.6)
- added U11: 74LVC2G08, Package_SO:VSSOP-8_2.3x2mm_P0.5mm, F.Cu at (25.9, 22.4)
- added U12: 74LVC2G86, Package_SO:VSSOP-8_2.3x2mm_P0.5mm, F.Cu at (25.9, 26.1)
- added U13: 74LVC2G08, Package_SO:VSSOP-8_2.3x2mm_P0.5mm, F.Cu at (25.9, 29.8)
- added U14: 74LVC2G08, Package_SO:VSSOP-8_2.3x2mm_P0.5mm, F.Cu at (25.9, 33.5)
- added U15: 74LVC2G32, Package_SO:VSSOP-8_2.3x2mm_P0.5mm, F.Cu at (25.9, 37.2)
- added U16: 74LVC2G32, Package_SO:VSSOP-8_2.3x2mm_P0.5mm, F.Cu at (25.9, 40.9)
- added U17: 74LVC2G86, Package_SO:VSSOP-8_2.3x2mm_P0.5mm, F.Cu at (25.9, 44.6)
- added U18: 74LVC2G86, Package_SO:VSSOP-8_2.3x2mm_P0.5mm, F.Cu at (25.9, 48.4)
- added U19: 74LVC2G86, Package_SO:VSSOP-8_2.3x2mm_P0.5mm, F.Cu at (146.2, 41.6)
- added U2: 74LVC2G08, Package_SO:VSSOP-8_2.3x2mm_P0.5mm, F.Cu at (20.3, 22.4)
- added U20: 74LVC2G86, Package_SO:VSSOP-8_2.3x2mm_P0.5mm, F.Cu at (146.2, 46.7)
- added U21: 74LVC2G08, Package_SO:VSSOP-8_2.3x2mm_P0.5mm, F.Cu at (142.5, 41.6)
- added U22: 74LVC2G08, Package_SO:VSSOP-8_2.3x2mm_P0.5mm, F.Cu at (142.5, 46.7)
- added U23: 74LVC2G08, Package_SO:VSSOP-8_2.3x2mm_P0.5mm, F.Cu at (31.5, 33.5)
- added U24: 74LVC2G08, Package_SO:VSSOP-8_2.3x2mm_P0.5mm, F.Cu at (31.5, 37.2)
- added U25: 74LVC2G02, Package_SO:VSSOP-8_2.3x2mm_P0.5mm, F.Cu at (31.5, 40.9)
- added U26: 74LVC2G02, Package_SO:VSSOP-8_2.3x2mm_P0.5mm, F.Cu at (31.5, 44.6)
- added U27: 74LVC2G08, Package_SO:VSSOP-8_2.3x2mm_P0.5mm, F.Cu at (31.5, 48.4)
- added U28: 74LVC1G08, Package_TO_SOT_SMD:SOT-23-5, F.Cu at (60.5, 71.6)
- added U3: 74LVC2G08, Package_SO:VSSOP-8_2.3x2mm_P0.5mm, F.Cu at (20.3, 26.1)
- added U31: 74LVC1G332, Package_TO_SOT_SMD:SOT-23-6, F.Cu at (60.5, 76.3)
- added U32: 74LVC1G332, Package_TO_SOT_SMD:SOT-23-6, F.Cu at (60.5, 80.9)
- added U33: 74LVC1G332, Package_TO_SOT_SMD:SOT-23-6, F.Cu at (65.7, 71.6)
- added U34: 74LVC1G332, Package_TO_SOT_SMD:SOT-23-6, F.Cu at (65.7, 76.3)
- added U35: 74LVC1G332, Package_TO_SOT_SMD:SOT-23-6, F.Cu at (65.7, 80.9)
- added U36: 74LVC1G332, Package_TO_SOT_SMD:SOT-23-6, F.Cu at (70.8, 71.6)
- added U37: 74LVC1G332, Package_TO_SOT_SMD:SOT-23-6, F.Cu at (70.8, 76.3)
- added U38: 74LVC1G332, Package_TO_SOT_SMD:SOT-23-6, F.Cu at (70.8, 80.9)
- added U39: 74LVC2G86, Package_SO:VSSOP-8_2.3x2mm_P0.5mm, F.Cu at (37.1, 18.6)
- added U4: 74LVC2G08, Package_SO:VSSOP-8_2.3x2mm_P0.5mm, F.Cu at (20.3, 29.8)
- added U40: 74LVC2G86, Package_SO:VSSOP-8_2.3x2mm_P0.5mm, F.Cu at (37.1, 22.4)
- added U41: 74LVC2G86, Package_SO:VSSOP-8_2.3x2mm_P0.5mm, F.Cu at (37.1, 26.1)
- added U42: 74LVC2G86, Package_SO:VSSOP-8_2.3x2mm_P0.5mm, F.Cu at (37.1, 29.8)
- added U43: 74LVC2G86, Package_SO:VSSOP-8_2.3x2mm_P0.5mm, F.Cu at (37.1, 33.5)
- added U44: 74LVC2G86, Package_SO:VSSOP-8_2.3x2mm_P0.5mm, F.Cu at (37.1, 37.2)
- added U45: 74LVC2G86, Package_SO:VSSOP-8_2.3x2mm_P0.5mm, F.Cu at (37.1, 40.9)
- added U46: 74LVC2G86, Package_SO:VSSOP-8_2.3x2mm_P0.5mm, F.Cu at (37.1, 44.6)
- added U47: 74LVC2G86, Package_SO:VSSOP-8_2.3x2mm_P0.5mm, F.Cu at (37.1, 48.4)
- added U48: 74LVC2G86, Package_SO:VSSOP-8_2.3x2mm_P0.5mm, F.Cu at (42.7, 18.6)
- added U49: 74LVC2G86, Package_SO:VSSOP-8_2.3x2mm_P0.5mm, F.Cu at (42.7, 22.4)
- added U5: 74LVC2G08, Package_SO:VSSOP-8_2.3x2mm_P0.5mm, F.Cu at (20.3, 33.5)
- added U50: 74LVC2G86, Package_SO:VSSOP-8_2.3x2mm_P0.5mm, F.Cu at (42.7, 26.1)
- added U51: 74LVC2G08, Package_SO:VSSOP-8_2.3x2mm_P0.5mm, F.Cu at (42.7, 29.8)
- added U52: 74LVC2G08, Package_SO:VSSOP-8_2.3x2mm_P0.5mm, F.Cu at (42.7, 33.5)
- added U53: 74LVC2G08, Package_SO:VSSOP-8_2.3x2mm_P0.5mm, F.Cu at (42.7, 37.2)
- added U54: 74LVC2G08, Package_SO:VSSOP-8_2.3x2mm_P0.5mm, F.Cu at (42.7, 40.9)
- added U55: 74LVC2G08, Package_SO:VSSOP-8_2.3x2mm_P0.5mm, F.Cu at (42.7, 44.6)
- added U56: 74LVC2G08, Package_SO:VSSOP-8_2.3x2mm_P0.5mm, F.Cu at (42.7, 48.4)
- added U57: 74LVC2G08, Package_SO:VSSOP-8_2.3x2mm_P0.5mm, F.Cu at (48.4, 18.6)
- added U58: 74LVC2G08, Package_SO:VSSOP-8_2.3x2mm_P0.5mm, F.Cu at (48.4, 22.4)
- added U59: 74LVC2G08, Package_SO:VSSOP-8_2.3x2mm_P0.5mm, F.Cu at (48.4, 26.1)
- added U6: 74LVC2G86, Package_SO:VSSOP-8_2.3x2mm_P0.5mm, F.Cu at (20.3, 37.2)
- added U60: 74LVC2G08, Package_SO:VSSOP-8_2.3x2mm_P0.5mm, F.Cu at (48.4, 29.8)
- added U61: 74LVC2G08, Package_SO:VSSOP-8_2.3x2mm_P0.5mm, F.Cu at (48.4, 33.5)
- added U62: 74LVC2G08, Package_SO:VSSOP-8_2.3x2mm_P0.5mm, F.Cu at (48.4, 37.2)
- added U7: 74LVC2G32, Package_SO:VSSOP-8_2.3x2mm_P0.5mm, F.Cu at (20.3, 40.9)
- added U8: 74LVC2G32, Package_SO:VSSOP-8_2.3x2mm_P0.5mm, F.Cu at (20.3, 44.6)
- added U9: 74LVC2G86, Package_SO:VSSOP-8_2.3x2mm_P0.5mm, F.Cu at (20.3, 48.4)
Routing:
- net A2: track 0.00 -> 45.7 mm, vias 0 -> 2
- net A0: track 0.00 -> 32.4 mm
- net A1: track 0.00 -> 24.4 mm, vias 0 -> 2
- net A3: track 0.00 -> 19.9 mm, vias 0 -> 2
- net B2: track 0.00 -> 12.8 mm, vias 0 -> 1
- net B1: track 0.00 -> 12.1 mm, vias 0 -> 1
- net B0: track 0.00 -> 11.8 mm, vias 0 -> 1
- net B3: track 0.00 -> 9.90 mm, vias 0 -> 1
- net GND: track 0.00 -> 4.17 mm, vias 0 -> 4
- net XOR3: track 0.00 -> 3.04 mm, vias 0 -> 1
- net +3V0: track 0.00 -> 2.91 mm, vias 0 -> 3
- net XOR1: track 0.00 -> 2.86 mm, vias 0 -> 1
- net AND1: track 0.00 -> 2.56 mm, vias 0 -> 1
- net XOR0: track 0.00 -> 2.46 mm, vias 0 -> 1
- net AND3: track 0.00 -> 2.38 mm, vias 0 -> 1
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