File: ALU.kicad_sch (KiCad schematic)
At the start: 20 parts, among them SW3 SW_DIP_x08, SW4 SW_DIP_x08, U1 4070, U2 74LVC2G08, U3 74LVC2G08, U4 74LVC2G08, U5 74LVC2G08, U6 4070, U7 74LVC2G32, U8 74LVC2G32

Commit message: Subtraction and logical operations
hmmm yes tasty

Total work time: 5.5 hours
Parts:
- added Ce3, Ce4, Ce5, Ce6, Ce7: 200n, symbol Device:C_Polarized
- added R10, R11, R12, R13, R14, R15, R16, R9: 10K, symbol Device:R
- added U10, U11, U13, U14, U21, U22, U23, U24: 74LVC2G08, symbol 74xGxx:74LVC2G08
- added U12, U17, U18, U19, U20, U9: 4070, symbol 4xxx:4070
- added U15, U16: 74LVC2G32, symbol 74xGxx:74LVC2G32
Connections:
- net +5V: now also Ce3.1, Ce4.1, Ce6.1, Ce7.1, U10.8 (VCC), U11.4 (GND), U12.14 (VDD), U13.8 (VCC), U14.4 (GND), U15.8 (VCC), U16.8 (VCC), U17.14 (VDD), U19.14 (VDD), U20.14 (VDD), U21.8 (VCC), U22.4 (GND), U23.8 (VCC), U24.8 (VCC), U9.14 (VDD)
- net A0: now also U1.1, U2.1, U19.1
- net A1: now also U1.5, U2.5, U19.5
- net A2: now also U1.8, U3.1, U19.8
- net A3: now also U1.12, U3.5, U19.12
- net A4: now also SW3.12, R9.2, U10.1, U20.1, U9.1
- net A5: now also SW3.11, R10.2, U10.5, U20.5, U9.5
- net A6: now also SW3.10, R11.2, U11.1, U20.8, U9.8
- net A7: now also SW3.9, R12.2, U11.5, U20.12, U9.12
- net B0: now also U17.1, U19.2
- net B1: now also U17.5, U19.6
- net B2: now also U17.8, U19.9
- net B3: now also U17.12, U19.13
- net B4: now also SW4.12, R13.2, U18.1, U20.2
- net B5: now also SW4.11, R14.2, U18.5, U20.6
- net B6: now also SW4.10, R15.2, U18.8, U20.9
- net B7: now also SW4.9, R16.2, U18.12, U20.13
- net C1: now also U5.5, U6.5
- net C1A: now also U7.1
- net C1B: now also U7.2
- net C2: now also U4.1, U6.8
- net C2A: now also U7.5
- net C2B: now also U7.6
- net C3: now also U4.5, U6.12
- net C3A: now also U8.1
- net C3B: now also U8.2
- net C4: now also U12.1, U13.1
- net C4A: now also U8.5
- net C4B: now also U8.6
- net CIN: now also U5.1, U6.1
- net GND: now also Ce3.2, Ce4.2, Ce5.2, Ce6.2, Ce7.2, R10.1, R11.1, R12.1, R13.1, R14.1, R15.1, R16.1, R9.1, U10.4 (GND), U11.8 (VCC), U12.7 (VSS), U13.4 (GND), U14.8 (VCC), U15.4 (GND), U16.4 (GND), U17.7 (VSS), U18.7 (VSS), U19.7 (VSS), U20.7 (VSS), U21.4 (GND), U22.8 (VCC), U23.4 (GND), U24.4 (GND), U9.7 (VSS)
- net S0A: now also U5.2, U6.2
- net S1A: now also U5.6, U6.6
- net S2A: now also U4.2, U6.9
- net S3A: now also U4.6, U6.13
- net at U3.6: now also U1.13, U17.11
- net at U1.6: now also U2.6, U17.4
- net at U2.2: now also U1.2, U17.3
- net at U1.9: now also U3.2, U17.10
- new net: Ce5.1, U18.14 (VDD)
- new net: U11.6, U18.11, U9.13
- new net: U11.2, U18.10, U9.9
- new net: U10.6, U18.4, U9.6
- new net: U10.2, U18.3, U9.2
- new net !B: U17.13, U17.2, U17.6, U17.9, U18.13, U18.2, U18.6, U18.9
- new net C5: U12.5, U13.5, U15.7
- new net C5A: U10.7, U15.1
- new net C5B: U13.7, U15.2
- new net C6: U12.8, U14.1, U15.3
- new net C6A: U10.3, U15.5
- new net C6B: U13.3, U15.6
- new net C7: U12.12, U14.5, U16.7
- new net C7A: U11.7, U16.1
- new net C7B: U14.7, U16.2
- new net C8A: U11.3, U16.5
- new net C8B: U14.3, U16.6
- new net COUT: U16.3
- new net S4: U12.3
- new net S4A: U12.2, U13.2, U9.3
- new net S5: U12.4
- new net S5A: U12.6, U13.6, U9.4
- new net S6: U12.10
- new net S6A: U12.9, U14.2, U9.10
- new net S7: U12.11
- new net S7A: U12.13, U14.6, U9.11
Other:
- moved on the sheet: Ce1, Ce2, R1, R2, R3, R4, R5, R6, R7, R8, U1A, U1B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

Commit message: mux and stuff
6.6 hours work time
Parts:
- added Ce8: 200n, symbol Device:C_Polarized
- added U25, U26, U27, U28, U29, U30: 74LS09, symbol 74xx:74LS09
- added U31, U32, U33, U34, U35, U36, U37, U38: 74LVC1G332, symbol 74xGxx:74LVC1G332
- added U39, U40: 4070, symbol 4xxx:4070
Connections:
- net +5V: now also Ce8.1, U25.14 (VCC), U26.14 (VCC), U27.14 (VCC), U28.14 (VCC), U29.14 (VCC), U30.14 (VCC), U39.14 (VDD), U40.14 (VDD)
- net A0: now also U21.1
- net A1: now also U21.5
- net A2: now also U22.1
- net A3: now also U22.5
- net A4: now also U23.1
- net A5: now also U23.5
- net A6: now also U24.1
- net A7: now also U24.5
- net B0: now also U21.2
- net B1: now also U21.6
- net B2: now also U22.2
- net B3: now also U22.6
- net B4: now also U23.2
- net B5: now also U23.6
- net B6: now also U24.2
- net B7: now also U24.6
- net GND: now also Ce8.2, U25.7 (GND), U26.7 (GND), U27.7 (GND), U28.7 (GND), U29.7 (GND), U30.7 (GND), U31.2 (GND), U32.2 (GND), U33.2 (GND), U34.2 (GND), U35.2 (GND), U36.2 (GND), U37.2 (GND), U38.2 (GND), U39.7 (VSS), U40.7 (VSS)
- net S0: now also U29.1
- net S1: now also U29.4
- net S2: now also U29.9
- net S3: now also U29.12
- net S4: now also U30.1
- net S5: now also U30.4
- net S6: now also U30.9
- net S7: now also U30.12
- net AND3: now reaches U22.3
- net AND3: now also U25.12
- net XOR0: now reaches U19.3
- net XOR0: now also U27.1
- net AND7: now reaches U24.3
- net AND7: now also U26.12
- net XOR3: now reaches U19.11
- net XOR3: now also U27.12
- net XOR6: now reaches U20.10
- net XOR6: now also U28.9
- net AND2: now reaches U22.7
- net AND2: now also U25.9
- net AND0: now reaches U21.7
- net AND0: now also U25.1
- net XOR1: now reaches U19.4
- net XOR1: now also U27.4
- net XOR2: now reaches U19.10
- net XOR2: now also U27.9
- net AND5: now reaches U23.3
- net AND5: now also U26.4
- net XOR5: now reaches U20.4
- net XOR5: now also U28.4
- net AND1: now reaches U21.3
- net AND1: now also U25.4
- net AND4: now reaches U23.7
- net AND4: now also U26.1
- net AND6: now reaches U24.7
- net AND6: now also U26.9
- net XOR7: now reaches U20.11
- net XOR7: now also U28.12
- net XOR4: now reaches U20.3
- net XOR4: now also U28.1
- new net: U31.4, U39.1
- new net: U34.4, U39.12
- new net: U32.4, U39.5
- new net: U35.4, U40.1
- new net: U33.4, U39.8
- new net: U36.4, U40.5
- new net: U38.4, U40.12
- new net: U37.4, U40.8
- new net !O: U39.13, U39.2, U39.6, U39.9, U40.13, U40.2, U40.6, U40.9
- new net ENA_ADD: U29.10, U29.13, U29.2, U29.5, U30.10, U30.13, U30.2, U30.5
- new net ENA_AND: U25.10, U25.13, U25.2, U25.5, U26.10, U26.13, U26.2, U26.5
- new net ENA_XOR: U27.10, U27.13, U27.2, U27.5, U28.10, U28.13, U28.2, U28.5
- new net M_ADD0: U29.3, U31.3
- new net M_ADD1: U29.6, U32.3
- new net M_ADD2: U29.8, U33.3
- new net M_ADD3: U29.11, U34.3
- new net M_ADD4: U30.3, U35.3
- new net M_ADD5: U30.6, U36.3
- new net M_ADD6: U30.8, U37.3
- new net M_ADD7: U30.11, U38.3
- new net M_AND0: U25.3, U31.6
- new net M_AND1: U25.6, U32.6
- new net M_AND2: U25.8, U33.6
- new net M_AND3: U25.11, U34.6
- new net M_AND4: U26.3, U35.6
- new net M_AND5: U26.6, U36.6
- new net M_AND6: U26.8, U37.6
- new net M_AND7: U26.11, U38.6
- new net M_XOR0: U27.3, U31.1
- new net M_XOR1: U27.6, U32.1
- new net M_XOR2: U27.8, U33.1
- new net M_XOR3: U27.11, U34.1
- new net M_XOR4: U28.3, U35.1
- new net M_XOR5: U28.6, U36.1
- new net M_XOR6: U28.8, U37.1
- new net M_XOR7: U28.11, U38.1
Other:
- moved on the sheet: Ce7, U21A, U21B, U21C, U22A, U22B, U22C, U23A, U23B, U23C, U24A, U24B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

Commit message: Add files via upload
Parts:
- removed U1, U12, U17, U18, U19, U20, U39, U40, U6, U9: 4070, symbol 4xxx:4070
- removed U25, U26, U27, U28, U29, U30: 74LS09, symbol 74xx:74LS09
- added U1, U12, U17, U18, U19, U20, U39, U40, U41, U42, U43, U44, U45, U46, U47, U48, U49, U50, U6, U9: 74LVC2G86, symbol 74xGxx:74LVC2G86
- added U51, U52, U53, U54, U55, U56, U57, U58, U59, U60, U61, U62: 74LVC2G08, symbol 74xGxx:74LVC2G08
Connections:
- net !B: now also U41.2, U41.6, U42.2, U42.6, U43.2, U43.6, U44.2, U44.6
- net !O: now also U39.2, U39.6, U40.2, U40.6, U49.2, U49.6, U50.2, U50.6
- net +5V: now also Ce5.1, U11.8 (VCC), U14.8 (VCC), U2.8 (VCC), U31.5 (VCC), U32.5 (VCC), U33.5 (VCC), U34.5 (VCC), U35.5 (VCC), U36.5 (VCC), U37.5 (VCC), U38.5 (VCC), U5.8 (VCC), U1.8 (VCC), U17.8 (VCC), U18.8 (VCC), U19.8 (VCC), U20.8 (VCC), U39.8 (VCC), U40.8 (VCC), U41.8 (VCC), U42.8 (VCC), U43.8 (VCC), U44.8 (VCC), U45.8 (VCC), U46.8 (VCC), U47.8 (VCC), U48.8 (VCC), U49.8 (VCC), U50.8 (VCC), U53.8 (VCC), U54.8 (VCC), U55.8 (VCC), U56.8 (VCC), U57.8 (VCC), U58.8 (VCC), U59.8 (VCC), U60.8 (VCC), U61.8 (VCC), U62.8 (VCC), U9.8 (VCC); no longer U11.4 (GND), U14.4 (GND), U2.4 (GND), U5.4 (GND)
- net A0: now also U19.1, U9.1
- net A1: now also U19.5, U9.5
- net A2: now also U17.1, U20.1
- net A3: now also U17.5, U20.5
- net A4: now also U1.1, U47.1
- net A5: now also U1.5, U47.5
- net A6: now also U18.1, U48.1
- net A7: now also U48.5
- net AND0: now also U51.1
- net AND1: now also U51.5
- net AND2: now also U52.1
- net AND3: now also U52.5
- net AND4: now also U53.1
- net AND5: now also U53.5
- net AND6: now also U54.1
- net AND7: now also U54.5
- net B0: now also U19.2, U41.1
- net B1: now also U19.6, U41.5
- net B2: now also U20.2, U42.1
- net B3: now also U20.6, U42.5
- net B4: now also U43.1, U47.2
- net B5: now also U43.5, U47.6
- net B6: now also U44.1, U48.2
- net B7: now also U44.5, U48.6
- net C1: now also U6.5
- net C2: now also U12.1
- net C3: now also U12.5
- net C4: now also U45.1
- net C5: now also U45.5
- net C6: now also U46.1
- net C7: now also U46.5
- net C8A: no longer U11.3
- net CIN: now also U6.1
- net ENA_ADD: now also U59.2, U59.6, U60.2, U60.6, U61.2, U61.6, U62.2, U62.6
- net ENA_AND: now also U51.2, U51.6, U52.2, U52.6, U53.2, U53.6, U54.2, U54.6
- net ENA_XOR: now also U55.2, U55.6, U56.2, U56.6, U57.2, U57.6, U58.2, U58.6
- net GND: now also U11.4 (GND), U14.4 (GND), U2.4 (GND), U5.4 (GND), U1.4 (GND), U17.4 (GND), U18.4 (GND), U19.4 (GND), U20.4 (GND), U39.4 (GND), U40.4 (GND), U41.4 (GND), U42.4 (GND), U43.4 (GND), U44.4 (GND), U45.4 (GND), U46.4 (GND), U47.4 (GND), U48.4 (GND), U49.4 (GND), U50.4 (GND), U51.4 (GND), U52.4 (GND), U53.4 (GND), U54.4 (GND), U55.4 (GND), U56.4 (GND), U57.4 (GND), U58.4 (GND), U59.4 (GND), U60.4 (GND), U61.4 (GND), U62.4 (GND), U9.4 (GND); no longer U11.8 (VCC), U14.8 (VCC), U2.8 (VCC), U5.8 (VCC)
- net M_ADD0: now also U59.7
- net M_ADD1: now also U59.3
- net M_ADD2: now also U60.7
- net M_ADD3: now also U60.3
- net M_ADD4: now also U61.7
- net M_ADD5: now also U61.3
- net M_ADD6: now also U62.7
- net M_ADD7: now also U62.3
- net M_AND0: now also U51.7
- net M_AND1: now also U51.3
- net M_AND2: now also U52.7
- net M_AND3: now also U52.3
- net M_AND4: now also U53.7
- net M_AND5: now also U53.3
- net M_AND6: now also U54.7
- net M_AND7: now also U54.3
- net M_XOR0: now also U55.7
- net M_XOR1: now also U55.3
- net M_XOR2: now also U56.7
- net M_XOR3: now also U56.3
- net M_XOR4: now also U57.7
- net M_XOR5: now also U57.3
- net M_XOR6: now also U58.7
- net M_XOR7: now also U58.3
- net S0: now also U6.7
- net S0A: now also U6.2, U9.7
- net S1: now also U6.3
- net S1A: now also U6.6, U9.3
- net S2: now also U12.7
- net S2A: now also U12.2, U17.7
- net S3: now also U12.3
- net S3A: now also U12.6, U17.3
- net S4: now also U45.7
- net S4A: now also U1.7, U45.2
- net S5: now also U45.3
- net S5A: now also U1.3, U45.6
- net S6: now also U46.7
- net S6A: now also U18.7, U46.2
- net S7: now also U46.3
- net S7A: now also U46.6
- net XOR0: now also U19.7, U55.1
- net XOR1: now also U19.3, U55.5
- net XOR2: now also U20.7, U56.1
- net XOR3: now also U20.3, U56.5
- net XOR4: now also U47.7, U57.1
- net XOR5: now also U47.3, U57.5
- net XOR6: now also U48.7, U58.1
- net XOR7: now also U48.3, U58.5
- net at U3.6: now also U17.6, U42.3
- net at U31.4: now also U39.1
- net at U3.2: now also U17.2, U42.7
- net at U34.4: now also U40.5
- net at U11.6: now also U18.6, U44.3
- net at U32.4: now also U39.5
- net at U35.4: now also U49.1
- net at U33.4: now also U40.1
- net at U36.4: now also U49.5
- net at U2.2: now also U41.7, U9.2
- net at U2.6: now also U41.3, U9.6
- net at U11.2: now also U18.2, U44.7
- net at U10.6: now also U1.6, U43.3
- net at U38.4: now also U50.5
- net at U37.4: now also U50.1
- net at U10.2: now also U1.2, U43.7
- new net ADD0: U59.1
- new net ADD1: U59.5
- new net ADD2: U60.1
- new net ADD3: U60.5
- new net ADD4: U61.1
- new net ADD5: U61.5
- new net ADD6: U62.1
- new net ADD7: U62.5
Other:
- moved on the sheet: Ce1, Ce2, Ce3, Ce4, Ce5, Ce6, Ce7, Ce8, U10A, U10B, U10C, U11A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

Commit message: Revision 1.0!
9.2 hours work time
Parts:
- removed Ce1, Ce2, Ce3, Ce4, Ce5, Ce6, Ce7, Ce8: 200n, symbol Device:C_Polarized
- added BT1: 3V0, symbol Device:Battery_Cell
- added C1: 10u, symbol Device:C_Polarized
- added C10, C2, C3, C4, C5, C6, C7, C8, C9: 100n, symbol Device:C_Small
- added D1, D2, D3, D4, D5, D6, D7, D8: LED_GREEN, symbol Device:LED
- added D10, D9: LED_RED, symbol Device:LED
- added R17, R18, R19, R20, R21, R22: 10K, symbol Device:R
- added R23, R24, R25, R26, R27, R28, R29, R30, R31, R32, R33: 220, symbol Device:R
- added SW1: SW_DIP_x06, symbol Switch:SW_DIP_x06
- added SW2: SW_SPST_LED_YELLOW, symbol Switch:SW_SPST_LED
- added U25, U26: 74LVC2G02, symbol 74xGxx:74LVC2G02
- added U27: 74LVC2G08, symbol 74xGxx:74LVC2G08
- added U28: 74LVC1G08, symbol 74xGxx:74LVC1G08
Connections:
- net +5V is gone; now on net +3V0: SW3.1, SW3.2, SW3.3, SW3.4, SW3.5, SW3.6, SW3.7, SW3.8, SW4.1, SW4.2, SW4.3, SW4.4, SW4.5, SW4.6, SW4.7, SW4.8, U1.8 (VCC), U10.8 (VCC), U11.8 (VCC), U13.8 (VCC), U14.8 (VCC), U15.8 (VCC), U16.8 (VCC), U17.8 (VCC), U18.8 (VCC), U19.8 (VCC), U2.8 (VCC), U20.8 (VCC), U21.8 (VCC), U22.4 (GND), U23.8 (VCC), U24.8 (VCC), U3.8 (VCC), U31.5 (VCC), U32.5 (VCC), U33.5 (VCC), U34.5 (VCC), U35.5 (VCC), U36.5 (VCC), U37.5 (VCC), U38.5 (VCC), U39.8 (VCC), U4.8 (VCC), U40.8 (VCC), U41.8 (VCC), U42.8 (VCC), U43.8 (VCC), U44.8 (VCC), U45.8 (VCC), U46.8 (VCC), U47.8 (VCC), U48.8 (VCC), U49.8 (VCC), U5.8 (VCC), U50.8 (VCC), U53.8 (VCC), U54.8 (VCC), U55.8 (VCC), U56.8 (VCC), U57.8 (VCC), U58.8 (VCC), U59.8 (VCC), U60.8 (VCC), U61.8 (VCC), U62.8 (VCC), U7.8 (VCC), U8.8 (VCC), U9.8 (VCC)
- net !B: now also R20.2, SW1.9
- net !O: now also R21.2, SW1.8
- net CIN: now also R22.2, SW1.7
- net COUT: now also D9.2 (A)
- net ENA_ADD: now also R17.2, SW1.12
- net ENA_AND: now also R18.2, SW1.11
- net ENA_XOR: now also R19.2, SW1.10
- net GND: now also U12.4 (GND), U6.4 (GND), C1.2, C10.2, C2.2, C3.2, C4.2, C5.2, C6.2, C7.2, C8.2, C9.2, R17.1, R18.1, R19.1, R20.1, R21.1, R22.1, R24.2, R25.2, R26.2, R27.2, R28.2, R29.2, R30.2, R31.2, R32.2, R33.2, SW2.3 (K), U25.4 (GND), U26.4 (GND), U27.4 (GND), U28.3 (GND)
- net OUT1: now reaches U39.3
- net OUT1: now also D2.2 (A), U25.2
- net OUT6: now reaches U50.7
- net OUT6: now also D7.2 (A), U26.5
- net +3V0: now reaches U12.8 (VCC)
- net +3V0: now also U51.8 (VCC), U52.8 (VCC), U6.8 (VCC), C1.1, C10.1, C2.1, C3.1, C4.1, C5.1, C6.1, C7.1, C8.1, C9.1, R23.2, SW1.1, SW1.2, SW1.3, SW1.4, SW1.5, SW1.6, SW2.2, U25.8 (VCC), U26.8 (VCC), U27.8 (VCC), U28.5 (VCC)
- net OUT0: now reaches U39.7
- net OUT0: now also D1.2 (A), U25.1
- net OUT2: now reaches U40.7
- net OUT2: now also D3.2 (A), U25.5
- net OUT5: now reaches U49.3
- net OUT5: now also D6.2 (A), U26.2
- net OUT3: now reaches U40.3
- net OUT3: now also D4.2 (A), U25.6
- net OUT4: now reaches U49.7
- net OUT4: now also D5.2 (A), U26.1
- net OUT7: now reaches U50.3
- net OUT7: now also D8.2 (A), U26.6
- new net: BT1.1 (+), SW2.1
- new net: D2.1 (K), R25.1
- new net: D3.1 (K), R26.1
- new net: D4.1 (K), R27.1
- new net: D7.1 (K), R30.1
- new net: D8.1 (K), R31.1
- new net: U25.7, U27.5
- new net: U25.3, U27.6
- new net: D1.1 (K), R24.1
- new net: D10.1 (K), R33.1
- new net: D6.1 (K), R29.1
- new net: D5.1 (K), R28.1
- new net: D9.1 (K), R32.1
- new net: U26.3, U27.2
- new net: U26.7, U27.1
- new net: R23.1, SW2.4 (A)
- new net: U27.7, U28.2
- new net ZF: D10.2 (A), U28.4
Other:
- moved on the sheet: U10C, U11C, U12C, U13C, U14C, U15C, U16C, U17C, U18C, U19A, U19B, U19C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

Commit message: Revision 2.0 - Decoupling capacitors + Footprints
11.1 hours work time
Parts:
- added C11, C12, C13, C14, C15, C16, C17, C18, C19, C20, C21, C22, C23, C24, C25, C26, C27, C28, C29, C30, C31, C32, C33, C34, C35, C36, C37, C38, C39, C40, C41, C42, C43, C44, C45, C46, C47, C48, C49, C50, C51, C52, C53, C54, C55, C57, C58, C59, C60, C61: 100n, Capacitor_SMD:C_0805_2012Metric, symbol Device:C_Small
- BT1: footprint (none) -> Battery:Battery_Panasonic_CR2032-VS1N_Vertical_CircularHoles
- C1: footprint (none) -> Capacitor_THT:CP_Radial_D5.0mm_P2.00mm
- C10, C2, C3, C4, C5, C6, C7, C8, C9: footprint (none) -> Capacitor_SMD:C_0805_2012Metric
- D1, D10, D2, D3, D4, D5, D6, D7, D8, D9: footprint (none) -> LED_SMD:LED_0805_2012Metric
- R1, R10, R11, R12, R13, R14, R15, R16, R17, R18, R19, R2, R20, R21, R22, R24, R25, R26, R27, R28, R29, R3, R30, R31, R4, R5, R6, R7, R8, R9: footprint (none) -> Resistor_SMD:R_0805_2012Metric
- R23: value 220 -> 680; footprint (none) -> Resistor_SMD:R_0805_2012Metric
- R32, R33: value 220 -> 470; footprint (none) -> Resistor_SMD:R_0805_2012Metric
- SW1: footprint (none) -> Button_Switch_THT:SW_DIP_SPSTx06_Slide_9.78x17.42mm_W7.62mm_P2.54mm
- SW2: footprint (none) -> LED_SMD:LED_0603_1608Metric
- SW3, SW4: footprint (none) -> Button_Switch_THT:SW_DIP_SPSTx08_Slide_9.78x22.5mm_W7.62mm_P2.54mm
- U1, U10, U11, U12, U13, U14, U15, U16, U17, U18, U19, U2, U20, U21, U22, U23, U24, U25, U26, U27, U28, U3, U39, U4, U40, U41, U42, U43, U44, U45, U46, U47, U48, U49, U5, U50, U51, U52, U53, U54, U55, U56, U57, U58, U59, U6, U60, U61, U62, U7, U8, U9: footprint (none) -> Package_SO:VSSOP-8_2.3x2mm_P0.5mm
- U31, U32, U33, U34, U35, U36, U37, U38: footprint (none) -> Package_TO_SOT_SMD:SOT-23-6
Connections:
- net ADD0 is gone; now on net S0: U59.1
- net ADD1 is gone; now on net S1: U59.5
- net ADD2 is gone; now on net S2: U60.1
- net ADD3 is gone; now on net S3: U60.5
- net ADD4 is gone; now on net S4: U61.1
- net ADD5 is gone; now on net S5: U61.5
- net ADD6 is gone; now on net S6: U62.1
- net ADD7 is gone; now on net S7: U62.5
- net +3V0: now also C3.2, C4.2, C5.2, C6.2, C7.2, C8.2, U22.8 (VCC), C11.2, C12.2, C13.2, C14.2, C15.2, C16.2, C17.2, C18.2, C19.2, C20.2, C21.2, C22.2, C23.2, C24.2, C25.2, C26.2, C27.2, C28.2, C29.2, C30.2, C31.2, C32.2, C33.2, C34.2, C35.2, C36.2, C37.2, C38.2, C39.2, C40.2, C41.2, C42.2, C43.2, C44.2, C45.2, C46.2, C47.2, C48.2, C49.2, C50.2, C51.2, C52.2, C53.2, C54.2, C55.2, C57.1, C58.1, C59.1, C60.1, C61.1; no longer C3.1, C4.1, C5.1, C6.1, C7.1, C8.1, U22.4 (GND)
- net A7: now also U18.5
- net C8A: now also U11.3
- net GND: now also BT1.2 (-), C3.1, C4.1, C5.1, C6.1, C7.1, C8.1, U22.4 (GND), C11.1, C12.1, C13.1, C14.1, C15.1, C16.1, C17.1, C18.1, C19.1, C20.1, C21.1, C22.1, C23.1, C24.1, C25.1, C26.1, C27.1, C28.1, C29.1, C30.1, C31.1, C32.1, C33.1, C34.1, C35.1, C36.1, C37.1, C38.1, C39.1, C40.1, C41.1, C42.1, C43.1, C44.1, C45.1, C46.1, C47.1, C48.1, C49.1, C50.1, C51.1, C52.1, C53.1, C54.1, C55.1, C57.2, C58.2, C59.2, C60.2, C61.2; no longer C3.2, C4.2, C5.2, C6.2, C7.2, C8.2, U22.8 (VCC)
- net S7A: now also U18.3
- net at U27.3: now also U28.1
Other:
- moved on the sheet: U12C, U18B, U19C, U20C, U21C, U22C, U23C, U24C, U25C, U26C, U27C, U39C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

Commit message: pcb layout start (attempt 3)
15.3 hours work time
Parts:
- removed SW2: SW_SPST_LED_YELLOW, LED_SMD:LED_0603_1608Metric, symbol Switch:SW_SPST_LED
- added D11: LED_YELLOW, LED_SMD:LED_0603_1608Metric, symbol Device:LED
- added SW2: SW_SPST, Button_Switch_THT:SW_DIP_SPSTx01_Slide_9.78x4.72mm_W7.62mm_P2.54mm, symbol Switch:SW_SPST
- U28: footprint Package_SO:VSSOP-8_2.3x2mm_P0.5mm -> Package_TO_SOT_SMD:SOT-23-5
Connections:
- net +3V0: now also SW2.2 (B)
- net GND: now also D11.1 (K)
- net at BT1.1 (+): now also SW2.1 (A)
- net at R23.1: now also D11.2 (A)
Changed lines of the file:
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@@
 	(wire
 		(pts
+			(xy 29.21 252.73) (xy 31.75 252.73)
+		)
+		(stroke
+			(width 0)
+			(type default)
+		)
+	)
+	(wire
+		(pts
 			(xy 468.63 257.81) (xy 468.63 269.24)
 		)
@@
 	)
 	(symbol
+		(lib_id "Switch:SW_SPST")
+		(at 34.29 250.19 0)
+		(unit 1)
+		(body_style 1)
+		(exclude_from_sim no)
+		(in_bom yes)
+		(on_board yes)
+		(in_pos_files yes)
+		(dnp no)
+		(property "Reference" "SW2"
+			(at 28.194 248.92 0)
+			(show_name no)
+			(do_not_autoplace no)
+			(effects
+				(font
+					(size 1.27 1.27)
+				)
+			)
+		)
+		(property "Value" "SW_SPST"
+			(at 43.18 248.92 0)
+			(show_name no)
+			(do_not_autoplace no)
+			(effects
+				(font
+					(size 1.27 1.27)
+				)
+			)
+		)
+		(property "Footprint" "Button_Switch_THT:SW_DIP_SPSTx01_Slide_9.78x4.72mm_W7.62mm_P2.54mm"
+			(at 34.29 250.19 0)
+			(hide yes)
+			(show_name no)
+			(do_not_autoplace no)
+			(effects
+				(font
+					(size 1.27 1.27)
+				)
+			)
+		)
+		(property "Datasheet" ""
+			(at 34.29 250.19 0)
+			(hide yes)
+			(show_name no)
+			(do_not_autoplace no)
+			(effects
+				(font
+					(size 1.27 1.27)
+				)
+			)
+		)
+		(property "Description" "Single Pole Single Throw (SPST) switch"
+			(at 34.29 250.19 0)
+			(hide yes)
+			(show_name no)
+			(do_not_autoplace no)
+			(effects
+				(font
+					(size 1.27 1.27)
+				)
+			)
+		)
+		(pin "1"
+		)
+		(pin "2"
+		)
+		(instances
+			(project "ALU"
+				(path "/d7e53033-95e0-4649-ad5b-f44d59ca154e"
+					(reference "SW2")
+					(unit 1)
+				)
+			)
+		)
+	)
+	(symbol
 		(lib_id "Device:R")
 		(at 71.12 22.86 0)
@@
 			)
 		)
-		(property "Footprint" "Package_SO:VSSOP-8_2.3x2mm_P0.5mm"
+		(property "Footprint" "Package_TO_SOT_SMD:SOT-23-5"
 			(at 450.85 92.71 0)
 			(hide yes)
@@
 	(symbol
 		(lib_id "Device:LED")
+		(at 35.56 252.73 0)
+		(unit 1)
+		(body_style 1)
+		(exclude_from_sim no)
+		(in_bom yes)
+		(on_board yes)
+		(in_pos_files yes)
+		(dnp no)
+		(property "Reference" "D11"
+			(at 34.798 255.27 0)
+			(show_name no)
+			(do_not_autoplace no)
+			(effects
+				(font
+					(size 1.27 1.27)
+				)
+			)
+		)
+		(property "Value" "LED_YELLOW"
+			(at 34.798 257.81 0)
+			(show_name no)
+			(do_not_autoplace no)
+			(effects
+				(font
+					(size 1.27 1.27)
+				)
+			)
+		)
+		(property "Footprint" "LED_SMD:LED_0603_1608Metric"
+			(at 35.56 252.73 0)
+			(hide yes)
+			(show_name no)
+			(do_not_autoplace no)
+			(effects
+				(font
+					(size 1.27 1.27)
+				)
+			)
+		)
+		(property "Datasheet" ""
+			(at 35.56 252.73 0)
+			(hide yes)
+			(show_name no)
+			(do_not_autoplace no)
+			(effects
+				(font
+					(size 1.27 1.27)
+				)
+			)
+		)
+		(property "Description" "Light emitting diode"
+			(at 35.56 252.73 0)
+			(hide yes)
+			(show_name no)
+			(do_not_autoplace no)
+			(effects
+				(font
+					(size 1.27 1.27)
+				)
+			)
+		)
+		(property "Sim.Pins" "1=K 2=A"
+			(at 35.56 252.73 0)
+			(hide yes)
+			(show_name no)
+			(do_not_autoplace no)
+			(effects
+				(font
+					(size 1.27 1.27)
+				)
+			)
+		)
+		(pin "1"
+		)
+		(pin "2"
+		)
+		(instances
+			(project "ALU"
+				(path "/d7e53033-95e0-4649-ad5b-f44d59ca154e"
+					(reference "D11")
+					(unit 1)
+				)
+			)
+		)
+	)
+	(symbol
+		(lib_id "Device:LED")
 		(at 508 72.39 180)
 		(unit 1)
@@
 					(unit 1)
 				)
-			)
-		)
-	)
-	(symbol
-		(lib_id "Switch:SW_SPST_LED")
-		(at 34.29 252.73 0)
-		(unit 1)
-		(body_style 1)
-		(exclude_from_sim no)
-		(in_bom yes)
-		(on_board yes)
-		(in_pos_files yes)
-		(dnp no)
-		(property "Reference" "SW2"
-			(at 34.29 256.286 0)
-			(show_name no)
-			(do_not_autoplace no)
-			(effects
-				(font
-					(size 1.27 1.27)
-				)
-			)
-		)
-		(property "Value" "SW_SPST_LED_YELLOW"
-			(at 34.29 258.826 0)
-			(show_name no)
-			(do_not_autoplace no)
-			(effects
-				(font
-					(size 1.27 1.27)
-				)
-			)
-		)
-		(property "Footprint" "LED_SMD:LED_0603_1608Metric"
-			(at 34.29 245.11 0)
-			(hide yes)
-			(show_name no)
-			(do_not_autoplace no)
-			(effects
-				(font
-					(size 1.27 1.27)
-				)
-			)
-		)
-		(property "Datasheet" ""
-			(at 34.29 259.08 0)
-			(hide yes)
-			(show_name no)
-			(do_not_autoplace no)
-			(effects
-				(font
-					(size 1.27 1.27)
-				)
-			)
-		)
-		(property "Description" "Single Pole Single Throw (SPST) switch with LED, generic"
-			(at 34.29 252.73 0)
-			(hide yes)
-			(show_name no)
-			(do_not_autoplace no)
-			(effects
-				(font
-					(size 1.27 1.27)
-				)
-			)
-		)
-		(pin "1"
-		)
-		(pin "2"
-		)
-		(pin "3"
-		)
-		(pin "4"
-		)
-		(instances
-			(project "ALU"
-				(path "/d7e53033-95e0-4649-ad5b-f44d59ca154e"
-					(reference "SW2")
-					(unit 1)
-				)
